Commit message: follow_turtlebot frontend final change

File: drone_assets/urdf/turtlebot3_waffle_pi_colored_plate.xacro (robot description, xacro)
@@ -5,5 +5,5 @@
     <xacro:include filename="$(find turtlebot3_description)/urdf/turtlebot3_waffle_pi.urdf.xacro" />
     <material name="green1">
-        <color rgba="0.0 0.8 0.0 1.0"/>
+        <texture filename="file://$(find drone_assets)/urdf/marker0.png" />
     </material>
     <link name="colored_plate">
@@ -17,5 +17,5 @@
     </link>
     <gazebo reference="colored_plate">
-        <material>Gazebo/Green</material>
+        <material>marker0</material>
     </gazebo>
     <joint name="base_to_colored_plate" type="fixed">

Commit message: back to previous turtlebot3

File: drone_assets/urdf/turtlebot3_waffle_pi_colored_plate.xacro (robot description, xacro)
@@ -5,5 +5,5 @@
     <xacro:include filename="$(find turtlebot3_description)/urdf/turtlebot3_waffle_pi.urdf.xacro" />
     <material name="green1">
-        <texture filename="file://$(find drone_assets)/urdf/marker0.png" />
+        <color rgba="0.0 0.8 0.0 1.0"/>
     </material>
     <link name="colored_plate">
@@ -17,5 +17,5 @@
     </link>
     <gazebo reference="colored_plate">
-        <material>marker0</material>
+        <material>Gazebo/Green</material>
     </gazebo>
     <joint name="base_to_colored_plate" type="fixed">
